Commit message: 2wr_urdf

File: catkin_ws/src/m2wr_description/urdf/m2wr.xacro (robot description, xacro)
@@ -58,22 +58,9 @@
     </visual>
   </link>
+  <!-- Right wheel-->
   <xacro:link_wheel name="link_right_wheel"/>
-  <joint name="joint_right_wheel" type="continuous">
-    <origin rpy="0 0 0" xyz="-0.05 0.15 0"/>
-    <child link="link_right_wheel"/>
-    <parent link="link_chassis"/>
-    <axis rpy="0 0 0" xyz="0 1 0"/>
-    <!-- Where the joint is going to rotate -->
-    <limit effort="10000" velocity="1000"/>
-    <joint_properties damping="1.0" friction="1.0"/>
-  </joint>
+  <xacro:joint_wheel name="joint_right_wheel" child_link="link_right_wheel" origin_xyz="-0.05 0.15 0"/>
+  <!-- Left wheel-->
   <xacro:link_wheel name="link_left_wheel"/>
-  <joint name="joint_left_wheel" type="continuous">
-    <origin rpy="0 0 0" xyz="-0.05 -0.15 0"/>
-    <child link="link_left_wheel"/>
-    <parent link="link_chassis"/>
-    <axis rpy="0 0 0" xyz="0 1 0"/>
-    <limit effort="10000" velocity="1000"/>
-    <joint_properties damping="1.0" friction="1.0"/>
-  </joint>
+  <xacro:joint_wheel name="joint_left_wheel" child_link="link_left_wheel" origin_xyz="-0.05 -0.15 0"/>
 </robot>

File: catkin_ws/src/m2wr_description/urdf/macros.xacro (robot description, xacro)
@@ -22,3 +22,14 @@
         </link>
     </macro>
+    <macro name="joint_wheel" params="name child_link origin_xyz">
+        <joint name="${name}" type="continuous">
+            <origin rpy="0 0 0" xyz="${origin_xyz}"/>
+            <child link="${child_link}"/>
+            <parent link="link_chassis"/>
+            <axis rpy="0 0 0" xyz="0 1 0"/>
+            <!-- Where the joint is going to rotate -->
+            <limit effort="10000" velocity="1000"/>
+            <joint_properties damping="1.0" friction="1.0"/>
+        </joint>
+    </macro>
 </robot>

Commit message: Laser Scanning

File: catkin_ws/src/m2wr_description/urdf/m2wr.xacro (robot description, xacro)
@@ -58,4 +58,32 @@
     </visual>
   </link>
+  <!-- Sensor Laser -->
+  <link name="sensor_laser">
+    <inertial>
+      <mass value="1"/>
+      <origin rpy="0 0 0" xyz="0 0 0"/>
+      <!-- Using a macro, need to put inside the macros.xacro file -->
+      <xacro:cylinder_inertia mass="1" r="0.05" l="0.1"/>
+    </inertial>
+    <visual>
+      <origin rpy="0 0 0" xyz="0 0 0"/>
+      <geometry>
+        <cylinder radius="0.05" length="0.1"/>
+      </geometry>
+      <material name="white"/>
+    </visual>
+    <collision>
+      <origin rpy="0 0 0" xyz="0 0 0"/>
+      <geometry>
+        <cylinder radius="0.05" length="0.1"/>
+      </geometry>
+    </collision>
+  </link>
+  <joint name="joint_sensor_laser" type="fixed">
+    <!-- Position of the laser in relation to the chassis -->
+    <origin rpy="0 0 0" xyz="0.15 0 0.05"/>
+    <parent link="link_chassis"/>
+    <child link="sensor_laser"/>
+  </joint>
   <!-- Right wheel-->
   <xacro:link_wheel name="link_right_wheel"/>

File: catkin_ws/src/m2wr_description/urdf/macros.xacro (robot description, xacro)
@@ -33,3 +33,7 @@
         </joint>
     </macro>
+    <macro name="cylinder_inertia" params="mass r l">
+        <inertia ixx="${mass*(3*r*r+l*l)/12}" ixy="0" ixz="0"
+                 iyy="${mass*(3*r*r+l*l)/12}" iyz="0" izz="${mass*(r*r)/2}"/>
+    </macro>
 </robot>
